File: DMX/MHCI-DMX/MHCI-DMX.kicad_sch (KiCad schematic)
At the start: 91 parts, among them J1 XLR_Male, J10 Conn_01x02, J11 Conn_01x02, J12 Conn_01x02, J13 Conn_01x02, J14 Conn_01x02, J15 Conn_01x02, J16 Conn_01x04, J17 Conn_01x08, J18 Conn_01x04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

Commit message: Adding 680R bias resistor network
Parts:
- added R6, R7: 680R, Resistor_SMD:R_0402_1005Metric, symbol Device:R_US
Connections:
- net +5V_ISO: now also R6.2
- net A: now also R6.1
- net B: now also R7.2
- net GND_DMX: now also R7.1
- net DMX_PASSTHROUGH: no longer names the net of D1.2 (A), JP7.1 (A), K1.1, Q1.3 (D)
Other:
- note added: "DMX RESISTORS Check if these are needed for receiving as well. Togglable terminator resistor Consider if we need the relay"
- moved on the sheet: D1, D4, J1, J19, J2, JP13, JP3, JP4, JP5, JP6, JP7, JP8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

Commit message: New screen
Parts:
- removed D10, D8: GREEN, LED_SMD:LED_0603_1608Metric, symbol Device:LED
- removed D7, D9: RED, LED_SMD:LED_0603_1608Metric, symbol Device:LED
- removed R12, R13: 300R, Resistor_SMD:R_0603_1608Metric, symbol Device:R_US
- removed U2: ~, Package_SO:TSSOP-8_3x3mm_P0.65mm, symbol MHCI:PCA9633
- removed U8: TXB0108PW, Package_SO:TSSOP-20_4.4x6.5mm_P0.65mm, symbol Logic_LevelTranslator:TXB0108PW
- added J20, J9: Conn_01x03, Connector_JST:JST_XH_B3B-XH-AM_1x03_P2.50mm_Vertical, symbol Connector_Generic:Conn_01x03
- added J21: Conn_01x04, Connector_JST:JST_XH_B4B-XH-AM_1x04_P2.50mm_Vertical, symbol Connector_Generic:Conn_01x04
- added U12: TCA9517ADGK, Package_SO:VSSOP-8_3x3mm_P0.65mm, symbol Logic_LevelTranslator:TCA9517ADGK
- added U2: TXS0108EPW, Package_SO:TSSOP-20_4.4x6.5mm_P0.65mm, symbol Logic_LevelTranslator:TXS0108EPW
- R10, R11: value 300R -> 4K7; LCSC C23025 -> C23162
Connections:
- net +3V3: now also U12.1 (VCCA), U12.5 (EN), U2.10 (OE), U2.2 (VCCA)
- net +5V: now also R10.1, R11.1, J21.1 (Pin_1), U12.8 (VCCB)
- net A_IN: now also J9.3 (Pin_3)
- net A_OUT: now also J20.3 (Pin_3)
- net B_IN: now also J9.2 (Pin_2)
- net B_OUT: now also J20.2 (Pin_2)
- net CTI_RESET: now also U2.7 (A6)
- net GND: now also J21.4 (Pin_4), U12.4 (GND), U2.11 (GND)
- net GND_DMX: now also J20.1 (Pin_1), J9.1 (Pin_1)
- net GPIO_X1: now also U2.4 (A3)
- net GPIO_X2: now also U2.5 (A4)
- net GPIO_X3: now also U2.6 (A5)
- net GPIO_X5: now also U2.8 (A7)
- net GPIO_X6: now also U2.9 (A8)
- net SCL: now also U12.2 (SCLA)
- net SCL_5: now also R11.2, J21.2 (Pin_2), U12.7 (SCLB)
- net SDA: now also U12.3 (SDAA)
- net SDA_5: now also R10.2, J21.3 (Pin_3), U12.6 (SDAB)
- net at R20.1: now also U2.14 (B6)
- net at R22.1: now also U2.12 (B8)
- net at R21.1: now also U2.13 (B7)
- net at R19.1: now also U2.15 (B5)
- net at R18.1: now also U2.16 (B4)
- net at R17.1: now also U2.17 (B3)
- net at JP15.2 (C): now also U2.19 (VCCB)
